Commit message: Perception, showcase demo and docs
Product registry without required barcodes, the identity escalation ladder (barcode, label text with an optional second reader, re-look guidance, needs-human), box products, proposals, lane stock and inventory, with pre-declared bounds, append-only splits and Wilson-interval results.

The showcase scene (textured, stocked shelf, packed randomly rotated back room) is the default demo and the only recorded video; launch and simulation speed-ups; the website perception section, results, figures and schematics.

File: ros_ws/src/restocker_description/urdf/gripper.xacro (robot description, xacro)
@@ -3,5 +3,103 @@
 <!-- SPDX-License-Identifier: MIT -->
 <robot xmlns:xacro="http://www.ros.org/wiki/xacro">
-  <xacro:macro name="restocker_gripper" params="prefix">
+  <!-- One finger's collision: finger.size_xyz_m tiled into finger.pad_rows equal rows along x
+       (spec M10 §11 D9). The union is exactly the finger box, so geometric consumers see the same
+       volume; each row is its own contact, which a single box is not under DART (no torsional
+       friction, §11.2 F13). This is the *planning* form; the simulation description replaces it
+       with compliant row links (§11 D10 item 3). -->
+  <xacro:macro name="restocker_finger_pad_rows" params="geometry row">
+    <xacro:if value="${row &lt; geometry.finger.pad_rows}">
+      <xacro:property name="row_height" value="${geometry.finger.size_xyz_m[0] / geometry.finger.pad_rows}"/>
+      <collision>
+        <origin
+          xyz="${geometry.finger.center_xyz_m[0] - 0.5 * geometry.finger.size_xyz_m[0] + (row + 0.5) * row_height} ${geometry.finger.center_xyz_m[1]} ${geometry.finger.center_xyz_m[2]}"
+          rpy="0 0 0"/>
+        <geometry>
+          <box size="${row_height} ${geometry.finger.size_xyz_m[1]} ${geometry.finger.size_xyz_m[2]}"/>
+        </geometry>
+      </collision>
+      <xacro:restocker_finger_pad_rows geometry="${geometry}" row="${row + 1}"/>
+    </xacro:if>
+  </xacro:macro>
+  <!-- Simulation description only (spec M10 §11 D10 item 3): the pad is 3.3 mm of 60 Shore A
+       silicone on the finger's inner face, so the finger body keeps the box minus that layer and
+       each pad row becomes its own link on a prismatic spring-damper joint along the pad normal.
+       At rest the body and the four rows occupy exactly the old finger box. inner_sign is -1 for
+       the left finger (its inner face is local -y) and +1 for the right one. -->
+  <xacro:macro name="restocker_finger_body_collision" params="geometry inner_sign">
+    <!-- The body stops behind the full depth of the pad-row spheres (one row height), not just the
+         3.3 mm layer: a product pressed 2-3 mm into the soft contact would otherwise reach the
+         rigid flat body, and the grip would be carried by a degenerate face contact instead of
+         the rows (measured at 80 N: most of the pad load went through the body). -->
+    <xacro:property name="row_depth" value="${geometry.finger.size_xyz_m[0] / geometry.finger.pad_rows}"/>
+    <xacro:property name="body_thickness" value="${geometry.finger.size_xyz_m[1] - row_depth}"/>
+    <collision>
+      <origin
+        xyz="${geometry.finger.center_xyz_m[0]} ${-inner_sign * 0.5 * row_depth} ${geometry.finger.center_xyz_m[2]}"
+        rpy="0 0 0"/>
+      <geometry>
+        <box size="${geometry.finger.size_xyz_m[0]} ${body_thickness} ${geometry.finger.size_xyz_m[2]}"/>
+      </geometry>
+    </collision>
+  </xacro:macro>
+  <xacro:macro name="restocker_compliant_pad_row" params="geometry prefix side row">
+    <xacro:if value="${row &lt; geometry.finger.pad_rows}">
+      <xacro:property name="row_height" value="${geometry.finger.size_xyz_m[0] / geometry.finger.pad_rows}"/>
+      <xacro:property name="pad_thickness" value="${geometry.finger.pad.thickness_m}"/>
+      <!-- The left finger's inner face is its local -y, the right finger's its local +y. -->
+      <xacro:property name="inner_sign" value="${-1 if side == 'left' else 1}"/>
+      <xacro:property name="row_x" value="${geometry.finger.center_xyz_m[0] - 0.5 * geometry.finger.size_xyz_m[0] + (row + 0.5) * row_height}"/>
+      <xacro:property name="row_y" value="${inner_sign * (0.5 * geometry.finger.size_xyz_m[1] - 0.5 * pad_thickness)}"/>
+      <xacro:property name="pad_link" value="${prefix}${side}_finger_pad_row_${row}"/>
+      <link name="${pad_link}">
+        <!-- A flat row, one row height deep: against the upright product cylinder it is a line
+             contact along the product axis whose normal is the pad normal. It is as deep as the
+             inset finger body behind it is thick (see restocker_finger_body_collision), so a 3 mm
+             press never reaches the box's back edges. Spheres were tried and rejected: the Bullet
+             sphere-to-cylinder-side test reports no contact until the overlap is ~2 mm, then
+             throws the product out, and a single rib pushes an off-centre product further off. -->
+        <collision name="${pad_link}_collision">
+          <origin
+            xyz="${row_x} ${inner_sign * (0.5 * geometry.finger.size_xyz_m[1] - 0.5 * row_height)} ${geometry.finger.center_xyz_m[2]}"
+            rpy="0 0 0"/>
+          <geometry>
+            <box size="${row_height} ${row_height} ${geometry.finger.size_xyz_m[2]}"/>
+          </geometry>
+        </collision>
+        <xacro:box_inertial
+          mass="${geometry.finger.pad.row_mass_kg}"
+          x="${row_height}"
+          y="${pad_thickness}"
+          z="${geometry.finger.size_xyz_m[2]}"
+          xyz="${row_x} ${row_y} ${geometry.finger.center_xyz_m[2]}" rpy="0 0 0"/>
+      </link>
+      <!-- The joint frame sits on the finger frame at rest, so spring_reference 0 is the
+           uncompressed pad and a positive displacement is compression (the axis points away from
+           the product). Every limit is physical (spec M10 section 11 D10 item 3): travel is
+           symmetric and generous so rest sits strictly inside it (the Card 057 M1 trap) and the
+           spring alone bounds it — the 3.3 mm layer cannot compress past its own thickness and the
+           bond keeps extension smaller still; effort is 500 N, the spring's own 222 N plus the
+           damping at the fastest the pad moves (1.71 m/s under a 40 N step), with 2x margin so
+           F14's clip can never engage; velocity is UNBOUNDED (-1), because a bonded pad has no
+           speed limit of its own — the jaw's 0.12 m/s copied here would be 14x too small for that
+           same step and DART enforces velocity limits as solver constraints that engage during
+           contact (sdformat maps a negative value to infinity; 0 would freeze the joint). The pad
+           row's mass is the silicone; the finger body keeps its own. -->
+      <joint name="${pad_link}_joint" type="prismatic">
+        <parent link="${prefix}${side}_finger"/>
+        <child link="${pad_link}"/>
+        <origin xyz="0 0 0" rpy="0 0 0"/>
+        <axis xyz="0 ${-inner_sign} 0"/>
+        <limit lower="-0.002" upper="0.002" effort="${geometry.finger.pad.effort_n}" velocity="-1"/>
+        <dynamics damping="${geometry.finger.pad.row_damping_n_s_per_m}"/>
+      </joint>
+      <gazebo reference="${pad_link}_joint">
+        <springReference>0</springReference>
+        <springStiffness>${geometry.finger.pad.row_stiffness_n_per_m}</springStiffness>
+      </gazebo>
+      <xacro:restocker_compliant_pad_row geometry="${geometry}" prefix="${prefix}" side="${side}" row="${row + 1}"/>
+    </xacro:if>
+  </xacro:macro>
+  <xacro:macro name="restocker_gripper" params="prefix compliant_pads:=false">
     <xacro:property name="geometry" value="${restocker_gripper_geometry}"/>
     <xacro:property name="body_size" value="${' '.join(str(value) for value in geometry.body.size_xyz_m)}"/>
@@ -61,8 +159,12 @@
         <material name="restocker_orange"/>
       </visual>
-      <collision>
-        <origin xyz="${finger_center}" rpy="0 0 0"/>
-        <geometry><box size="${finger_size}"/></geometry>
-      </collision>
+      <xacro:unless value="${compliant_pads}">
+        <xacro:restocker_finger_pad_rows geometry="${geometry}" row="0"/>
+      </xacro:unless>
+      <xacro:if value="${compliant_pads}">
+        <xacro:restocker_finger_body_collision geometry="${geometry}" inner_sign="-1"/>
+      </xacro:if>
+      <!-- The finger body keeps its own mass and box inertia (§11 D10's "unchanged" row); the pad
+           rows are the additional silicone, 4.9 g each. -->
       <xacro:box_inertial
         mass="${geometry.finger.mass_kg}"
@@ -86,8 +188,10 @@
         <material name="restocker_orange"/>
       </visual>
-      <collision>
-        <origin xyz="${finger_center}" rpy="0 0 0"/>
-        <geometry><box size="${finger_size}"/></geometry>
-      </collision>
+      <xacro:unless value="${compliant_pads}">
+        <xacro:restocker_finger_pad_rows geometry="${geometry}" row="0"/>
+      </xacro:unless>
+      <xacro:if value="${compliant_pads}">
+        <xacro:restocker_finger_body_collision geometry="${geometry}" inner_sign="1"/>
+      </xacro:if>
       <xacro:box_inertial
         mass="${geometry.finger.mass_kg}"
@@ -97,4 +201,8 @@
         xyz="${finger_center}" rpy="0 0 0"/>
     </link>
+    <xacro:if value="${compliant_pads}">
+      <xacro:restocker_compliant_pad_row geometry="${geometry}" prefix="${prefix}" side="left" row="0"/>
+      <xacro:restocker_compliant_pad_row geometry="${geometry}" prefix="${prefix}" side="right" row="0"/>
+    </xacro:if>
   </xacro:macro>
 </robot>

File: ros_ws/src/restocker_description/urdf/robot.xacro (robot description, xacro)
@@ -21,10 +21,12 @@
   <xacro:macro
     name="restocker_robot"
-    params="prefix joint_limits_parameters_file wrist_camera_sensor:=true">
+    params="prefix joint_limits_parameters_file wrist_camera_sensor:=true compliant_pads:=false">
     <xacro:restocker_rail prefix="${prefix}"/>
     <xacro:restocker_arm
       prefix="${prefix}"
       joint_limits_parameters_file="${joint_limits_parameters_file}"/>
-    <xacro:restocker_gripper prefix="${prefix}"/>
+    <!-- compliant_pads is the simulation description's D10 form of the finger pad; the planning
+         and visualization descriptions keep D9's plain tiled collisions. -->
+    <xacro:restocker_gripper prefix="${prefix}" compliant_pads="${compliant_pads}"/>
     <xacro:restocker_wrist_camera prefix="${prefix}" sensor="${wrist_camera_sensor}"/>
     <xacro:restocker_beanie prefix="${prefix}" parent="${prefix}shoulder_link"/>
@@ -32,5 +34,5 @@
   <xacro:macro
     name="restocker_robot_with_parent"
-    params="prefix parent joint_limits_parameters_file wrist_camera_sensor:=true *origin">
+    params="prefix parent joint_limits_parameters_file wrist_camera_sensor:=true compliant_pads:=false *origin">
     <joint name="${prefix}rail_base_mount_joint" type="fixed">
       <parent link="${parent}"/>
@@ -41,5 +43,6 @@
       prefix="${prefix}"
       joint_limits_parameters_file="${joint_limits_parameters_file}"
-      wrist_camera_sensor="${wrist_camera_sensor}"/>
+      wrist_camera_sensor="${wrist_camera_sensor}"
+      compliant_pads="${compliant_pads}"/>
   </xacro:macro>
 </robot>

File: ros_ws/src/restocker_description/urdf/ros2_control.xacro (robot description, xacro)
@@ -3,8 +3,13 @@
 <!-- SPDX-License-Identifier: MIT -->
 <robot xmlns:xacro="http://www.ros.org/wiki/xacro">
-  <!-- Both command interfaces are exported for every joint; each controller claims one, decided
-       in controllers.yaml. The arm and rail use velocity feedforward, the gripper uses position.
-       The controller-manager post-limiter that rewrote velocity commands is disabled there. -->
-  <xacro:macro name="restocker_controlled_joint" params="name lower upper initial_position:=0.0">
+  <!-- Command interfaces are exported for every joint; each controller claims its own in
+       controllers.yaml. The arm and rail use velocity feedforward. The two finger joints also
+       export `effort`, which is the one their controller claims: spec M10 §11 D10 drives them as a
+       force-limited position controller (the position and velocity exports stay so the hardware
+       keeps the same state bookkeeping and hold_joints fallback). The controller-manager
+       post-limiter that rewrote velocity commands is disabled there. -->
+  <xacro:macro
+    name="restocker_controlled_joint"
+    params="name lower upper initial_position:=0.0 effort_command:=false">
     <joint name="${name}">
       <command_interface name="position">
@@ -13,4 +18,7 @@
       </command_interface>
       <command_interface name="velocity"/>
+      <xacro:if value="${effort_command}">
+        <command_interface name="effort"/>
+      </xacro:if>
       <state_interface name="position">
         <param name="initial_value">${initial_position}</param>
@@ -32,6 +40,6 @@
       <xacro:restocker_controlled_joint name="${prefix}wrist_2_joint" lower="${-2.0 * pi}" upper="${2.0 * pi}" initial_position="0.0"/>
       <xacro:restocker_controlled_joint name="${prefix}wrist_3_joint" lower="${-2.0 * pi}" upper="${2.0 * pi}" initial_position="0.0"/>
-      <xacro:restocker_controlled_joint name="${prefix}left_finger_joint" lower="${restocker_gripper_lower}" upper="${restocker_gripper_upper}" initial_position="0.005"/>
-      <xacro:restocker_controlled_joint name="${prefix}right_finger_joint" lower="${restocker_gripper_lower}" upper="${restocker_gripper_upper}" initial_position="0.005"/>
+      <xacro:restocker_controlled_joint name="${prefix}left_finger_joint" lower="${restocker_gripper_lower}" upper="${restocker_gripper_upper}" initial_position="0.005" effort_command="true"/>
+      <xacro:restocker_controlled_joint name="${prefix}right_finger_joint" lower="${restocker_gripper_lower}" upper="${restocker_gripper_upper}" initial_position="0.005" effort_command="true"/>
     </ros2_control>
     <gazebo>
@@ -39,7 +47,11 @@
         <parameters>${controller_config}</parameters>
         <hold_joints>true</hold_joints>
-        <!-- Position-commanded gripper only. At gain 1.0, post-release traverses repeatedly drove the
-             parked-open fingers past their hard bounds, and the impulses coincided with arm wrist
-             velocity-limit excursions. Gain 0.5 keeps short-stroke attachment accuracy without
+        <!-- Only ever applies to a *position*-claimed joint: gz_ros2_control turns that command
+             into v = -position_proportional_gain * (pos - cmd) * update_rate. No controller claims
+             one since the fingers moved to `effort` (spec M10 §11 D10 item 5), so this is inert
+             until something does — and note the slope is this gain times `update_rate`, which is
+             1000 Hz now, so it must be re-derived rather than reused if a position claim returns.
+             Its history: at gain 1.0 post-release traverses repeatedly drove the parked-open
+             fingers past their hard bounds; 0.5 kept short-stroke attachment accuracy without
              hammering those stops. -->
         <position_proportional_gain>0.5</position_proportional_gain>

File: ros_ws/src/restocker_gazebo/urdf/product.urdf.xacro (robot description, xacro)
@@ -5,4 +5,7 @@
   <xacro:arg name="radius" default="0.033"/>
   <xacro:arg name="height" default="0.122"/>
+  <!-- A box product (CMB-119) sets `box_size` to "x y z" metres (width, depth, height); radius and
+       height are then unused. Empty keeps the cylinder. -->
+  <xacro:arg name="box_size" default=""/>
   <xacro:arg name="mass" default="0.355"/>
   <xacro:arg name="rgba" default="0.78 0.12 0.08 1.0"/>
@@ -18,9 +21,21 @@
        against the Gazebo server's working directory. -->
   <xacro:arg name="label_texture" default=""/>
+  <!-- Absolute path to a visual-only mesh (a contoured bottle) drawn instead of the cylinder, or
+       empty. The collision is always the catalogue cylinder, so the mesh must sit inside it and
+       physics, grasp planning and the catalogue loaders never see the contour. -->
+  <xacro:arg name="visual_mesh" default=""/>
   <xacro:include filename="$(find restocker_description)/urdf/inertial_macros.xacro"/>
   <xacro:property name="product_radius" value="$(arg radius)"/>
   <xacro:property name="product_height" value="$(arg height)"/>
   <xacro:property name="product_mass" value="$(arg mass)"/>
+  <xacro:property name="box_size" value="$(arg box_size)"/>
+  <xacro:property name="is_box" value="${box_size != ''}"/>
+  <xacro:if value="${is_box}">
+    <xacro:property name="box_x" value="${float(box_size.split()[0])}"/>
+    <xacro:property name="box_y" value="${float(box_size.split()[1])}"/>
+    <xacro:property name="box_z" value="${float(box_size.split()[2])}"/>
+  </xacro:if>
   <xacro:property name="label_texture" value="$(arg label_texture)"/>
+  <xacro:property name="visual_mesh" value="$(arg visual_mesh)"/>
   <link name="product_body">
     <!-- The visual is named `product_body_visual` because sdformat's URDF parser only merges a
@@ -28,22 +43,50 @@
          `<link>_visual`. A visual named `product_visual` becomes
          `product_body_fixed_joint_lump__product_visual_visual`, the match fails, and the material
-         extension below is silently dropped (see `gz sdf -p`). The collision keeps its own name
-         deliberately; see the note on the extension block. -->
+         extension below is silently dropped (see `gz sdf -p`). The collision follows the same
+         rule: it must be `product_body_collision`, because that is the generated SDF name the
+         parser looks for when it merges `mu1`/`mu2`. It was named `product_collision` until
+         2026-09-29, so the friction never reached Gazebo; `test_simulation_description` now
+         asserts the converted SDF carries `<surface><friction>` for every shipped product. -->
     <visual name="product_body_visual">
-      <geometry><cylinder radius="${product_radius}" length="${product_height}"/></geometry>
+      <xacro:if value="${visual_mesh == '' and not is_box}">
+        <geometry><cylinder radius="${product_radius}" length="${product_height}"/></geometry>
+      </xacro:if>
+      <xacro:if value="${visual_mesh == '' and is_box}">
+        <geometry><box size="${box_x} ${box_y} ${box_z}"/></geometry>
+      </xacro:if>
+      <xacro:unless value="${visual_mesh == ''}">
+        <geometry><mesh filename="file://${visual_mesh}"/></geometry>
+      </xacro:unless>
       <material name="product_material"><color rgba="$(arg rgba)"/></material>
     </visual>
-    <collision name="product_collision">
-      <geometry><cylinder radius="${product_radius}" length="${product_height}"/></geometry>
+    <collision name="product_body_collision">
+      <xacro:unless value="${is_box}">
+        <geometry><cylinder radius="${product_radius}" length="${product_height}"/></geometry>
+      </xacro:unless>
+      <xacro:if value="${is_box}">
+        <geometry><box size="${box_x} ${box_y} ${box_z}"/></geometry>
+      </xacro:if>
     </collision>
-    <xacro:cylinder_inertial
-      mass="${product_mass}" radius="${product_radius}" length="${product_height}"
-      xyz="0 0 0" rpy="0 0 0"/>
+    <xacro:unless value="${is_box}">
+      <xacro:cylinder_inertial
+        mass="${product_mass}" radius="${product_radius}" length="${product_height}"
+        xyz="0 0 0" rpy="0 0 0"/>
+    </xacro:unless>
+    <xacro:if value="${is_box}">
+      <xacro:box_inertial
+        mass="${product_mass}" x="${box_x}" y="${box_y}" z="${box_z}" xyz="0 0 0" rpy="0 0 0"/>
+    </xacro:if>
   </link>
-  <!-- The friction and contact entries here have never reached Gazebo: sdformat drops them
-       because the collision is named `product_collision` and the parser looks for
-       `product_body_collision`. They are left as is because enabling them would change the
-       contact behaviour that every grasp, benchmark and attachment tolerance was measured
-       against. Renaming the collision is the whole fix. -->
+  <!-- These entries reach Gazebo as of 2026-09-29, once the collision above carries the name the
+       parser merges into. Only `mu1`/`mu2` do any work: DART's backend reads
+       `surface/friction/ode/mu` and combines it with the other body's by taking the smaller of
+       the two, so this value decides the contact whenever the other body's coefficient is at or
+       above it — the finger faces, the shelf (0.8) and the floor (0.9) all are — and the smaller
+       of two catalogued values decides product-to-product. `kp` and `kd` are emitted into
+       `surface/contact/ode` and then ignored: the DART backend never reads them (its contact
+       ERP/CFM are compiled in), so they are not a stiffness tuning surface and must not be
+       described as one. Before the rename the whole block was silently discarded, which is why
+       every grasp and attachment tolerance predating it has to be re-measured rather than cited
+       (Card 024). -->
   <gazebo reference="product_body">
     <mu1>$(arg friction)</mu1>
@@ -52,5 +95,6 @@
     <kd>1</kd>
     <xacro:unless value="${label_texture == ''}">
-      <!-- Gazebo unwraps a cylinder's lateral surface with u once around the circumference and v
+      <!-- (A box's texture is the face atlas its mesh's UVs index; see tools/generate_box_meshes.py.)
+           Gazebo unwraps a cylinder's lateral surface with u once around the circumference and v
            along the axis, so a plain image is enough for a label and no mesh is needed. The metal
            workflow with zero metalness gives matte paper; the default metalness renders a mirror

File: ros_ws/src/restocker_gazebo/urdf/restocker_sim.urdf.xacro (robot description, xacro)
@@ -11,8 +11,13 @@
        envelope, not a hardware torque rating. Keep that simulator-only setting out of the
        planning and visualization descriptions. -->
+  <!-- compliant_pads (spec M10 §11 D10 item 3) is the other simulator-only form: each finger pad
+       is 4 small links on prismatic spring-damper joints so the load is shared across the rows.
+       MoveIt plans against restocker_planning.urdf.xacro, which keeps D9's plain tiled
+       collisions and never sees these links. -->
   <xacro:restocker_robot
     prefix="$(arg prefix)"
     joint_limits_parameters_file="$(find restocker_description)/config/ur10e_sim_joint_limits.yaml"
-    wrist_camera_sensor="$(arg wrist_camera_sensor)"/>
+    wrist_camera_sensor="$(arg wrist_camera_sensor)"
+    compliant_pads="true"/>
   <xacro:restocker_ros2_control prefix="$(arg prefix)" controller_config="$(arg controller_config)"/>
 </robot>
